Commit message: Clean up code, use smaller params

File: obj_a.urdf (robot description, URDF)
Before this commit: robot UNNAMED_0, 1 links, 0 joints
Links:
- link obj_a: mass 100.0 -> 10.0; geometry collision box size=1.0 1.0 1.0; visual box size=1.0 1.0 1.0

File: obj_b.urdf (robot description, URDF)
Before this commit: robot UNNAMED_1, 1 links, 0 joints
Links:
- link obj_b: mass 60.0 -> 6.0; geometry collision box size=2.0 5.0 1.0; visual box size=2.0 5.0 1.0

File: obj_c.urdf (robot description, URDF)
Before this commit: robot UNNAMED_2, 1 links, 0 joints
Links:
- link obj_c: mass 300.5 -> 3.0; geometry collision box size=1.5 1.5 1.0; visual box size=1.5 1.5 1.0

File: obj_d.urdf (robot description, URDF)
Before this commit: robot UNNAMED_3, 1 links, 0 joints
Links:
- link obj_d: mass 150.0 -> 8.0
